File: display.kicad_pcb (KiCad board)
At the start: 2 copper layers, 18.8 x 27.9 mm, 14 parts, among them J1 Conn_02x06_Counter_Clockwise, J2 Conn_01x05_Female, J3 Conn_01x02_Female, SW1 SW_Push, U1 MDBT42Q

Commit message: update labels
Connections:
- net Net-(J2-Pad2) renamed /SWDIO
- net Net-(J2-Pad3) renamed /SWDCK
- net Net-(J2-Pad4) renamed /tRST
Other:
- board text added: "3V3"
- board text added: "GND"
- board text added: "RST"
- board text added: "SWDCK"
- board text added: "SWDIO"
Changed lines of the file:
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@@
   (general
     (thickness 0.8)
-    (drawings 6)
+    (drawings 13)
     (tracks 209)
     (zones 0)
@@
   (net 21 +3V3)
   (net 22 GND)
-  (net 23 "Net-(J2-Pad3)")
-  (net 24 "Net-(J2-Pad2)")
-  (net 25 "Net-(J2-Pad4)")
-  (net 26 "Net-(SW1-Pad1)")
+  (net 23 "Net-(SW1-Pad1)")
+  (net 24 /SWDIO)
+  (net 25 /SWDCK)
+  (net 26 /tRST)
   (net_class Default "This is the default net class."
     (clearance 0.2)
@@
     (add_net /K3)
     (add_net /K4)
+    (add_net /SWDCK)
+    (add_net /SWDIO)
+    (add_net /tRST)
     (add_net GND)
-    (add_net "Net-(J2-Pad2)")
-    (add_net "Net-(J2-Pad3)")
-    (add_net "Net-(J2-Pad4)")
     (add_net "Net-(R1-Pad1)")
     (add_net "Net-(R2-Pad1)")
@@
     (pad 38 smd rect (at 4.7 -2.9 180) (size 1.6 0.4) (layers F.Cu F.Paste F.Mask))
     (pad 37 smd rect (at 4.7 -2.2 180) (size 1.6 0.4) (layers F.Cu F.Paste F.Mask)
-      (net 24 "Net-(J2-Pad2)"))
+      (net 24 /SWDIO))
     (pad 36 smd rect (at 4.7 -1.5 180) (size 1.6 0.4) (layers F.Cu F.Paste F.Mask)
-      (net 23 "Net-(J2-Pad3)"))
+      (net 25 /SWDCK))
     (pad 35 smd rect (at 4.7 -0.8 180) (size 1.6 0.4) (layers F.Cu F.Paste F.Mask)
-      (net 25 "Net-(J2-Pad4)"))
+      (net 26 /tRST))
     (pad 34 smd rect (at 4.7 -0.1 180) (size 1.6 0.4) (layers F.Cu F.Paste F.Mask)
       (net 1 /K1))
@@
     (pad 14 smd rect (at -2.8 7.7 90) (size 1.6 0.4) (layers F.Cu F.Paste F.Mask))
     (pad 13 smd rect (at -3.5 7.7 90) (size 1.6 0.4) (layers F.Cu F.Paste F.Mask)
-      (net 26 "Net-(SW1-Pad1)"))
+      (net 23 "Net-(SW1-Pad1)"))
     (pad 41 smd rect (at 2.9 -1.85 180) (size 1 0.4) (layers F.Cu F.Paste F.Mask))
     (pad 40 smd rect (at 2.9 -3.25 180) (size 1 0.4) (layers F.Cu F.Paste F.Mask))
@@
     (fp_line (start -3 3.3) (end -3 -3.3) (layer F.Fab) (width 0.1))
     (pad 1 smd rect (at -3.975 -2.25) (size 1.55 1.3) (layers F.Cu F.Paste F.Mask)
-      (net 26 "Net-(SW1-Pad1)"))
+      (net 23 "Net-(SW1-Pad1)"))
     (pad 1 smd rect (at 3.975 -2.25) (size 1.55 1.3) (layers F.Cu F.Paste F.Mask)
-      (net 26 "Net-(SW1-Pad1)"))
+      (net 23 "Net-(SW1-Pad1)"))
     (pad 2 smd rect (at -3.975 2.25) (size 1.55 1.3) (layers F.Cu F.Paste F.Mask)
       (net 21 +3V3))
@@
       (net 21 +3V3))
     (pad 2 thru_hole oval (at 0 1 180) (size 0.85 0.85) (drill 0.5) (layers *.Cu *.Mask)
-      (net 24 "Net-(J2-Pad2)"))
+      (net 24 /SWDIO))
     (pad 3 thru_hole oval (at 0 2 180) (size 0.85 0.85) (drill 0.5) (layers *.Cu *.Mask)
-      (net 23 "Net-(J2-Pad3)"))
+      (net 25 /SWDCK))
     (pad 4 thru_hole oval (at 0 3 180) (size 0.85 0.85) (drill 0.5) (layers *.Cu *.Mask)
-      (net 25 "Net-(J2-Pad4)"))
+      (net 26 /tRST))
     (pad 5 thru_hole oval (at 0 4 180) (size 0.85 0.85) (drill 0.5) (layers *.Cu *.Mask)
       (net 22 GND))
@@
     (tags capacitor)
     (attr smd)
-    (fp_text reference C1 (at 0 -1.65 270) (layer F.SilkS)
+    (fp_text reference C1 (at 2.4 0) (layer F.SilkS)
       (effects (font (size 1 1) (thickness 0.15)))
     )
@@
       (rotate (xyz 0 0 0))
     )
+  )
+  (gr_text 3V3 (at 116.6 89.2 90) (layer F.SilkS)
+    (effects (font (size 0.6 0.6) (thickness 0.1)))
+  )
+  (gr_text GND (at 116.5 91.9 90) (layer F.SilkS)
+    (effects (font (size 0.6 0.6) (thickness 0.1)))
+  )
+  (gr_text 3V3 (at 115.6 85.4) (layer F.SilkS)
+    (effects (font (size 0.6 0.6) (thickness 0.1)))
+  )
+  (gr_text SWDIO (at 116.1 84.3) (layer F.SilkS)
+    (effects (font (size 0.6 0.6) (thickness 0.1)))
+  )
+  (gr_text SWDCK (at 116 83.5) (layer F.SilkS)
+    (effects (font (size 0.6 0.6) (thickness 0.1)))
+  )
+  (gr_text RST (at 115.6 82.4) (layer F.SilkS)
+    (effects (font (size 0.6 0.6) (thickness 0.1)))
+  )
+  (gr_text GND (at 115.7 81.3) (layer F.SilkS)
+    (effects (font (size 0.6 0.6) (thickness 0.1)))
   )
   (dimension 18.8 (width 0.3) (layer F.SilkS)
@@
   (segment (start 109.09 97.3) (end 108.89 97.1) (width 0.25) (layer F.Cu) (net 22))
   (segment (start 111 97.3) (end 109.09 97.3) (width 0.25) (layer F.Cu) (net 22))
-  (segment (start 111.849999 86.150001) (end 111.8 86.2) (width 0.25) (layer B.Cu) (net 23))
-  (segment (start 114.185001 86.150001) (end 111.849999 86.150001) (width 0.25) (layer B.Cu) (net 23))
-  (segment (start 114.250001 86.085001) (end 114.185001 86.150001) (width 0.25) (layer B.Cu) (net 23))
-  (segment (start 114.250001 84.039999) (end 114.250001 86.085001) (width 0.25) (layer B.Cu) (net 23))
-  (segment (start 113.139999 83.649999) (end 113.860001 83.649999) (width 0.25) (layer B.Cu) (net 23))
-  (segment (start 113.389998 83.4) (end 113.139999 83.649999) (width 0.25) (layer B.Cu) (net 23))
-  (segment (start 113.5 83.4) (end 113.389998 83.4) (width 0.25) (layer B.Cu) (net 23))
-  (via (at 111.8 86.2) (size 0.8) (drill 0.4) (layers F.Cu B.Cu) (net 23))
-  (segment (start 113.860001 83.649999) (end 114.250001 84.039999) (width 0.25) (layer B.Cu) (net 23))
-  (segment (start 110.18 86.2) (end 110.11 86.13) (width 0.25) (layer F.Cu) (net 23))
-  (segment (start 111.8 86.2) (end 110.18 86.2) (width 0.25) (layer F.Cu) (net 23))
+  (segment (start 111.849999 86.150001) (end 111.8 86.2) (width 0.25) (layer B.Cu) (net 25))
+  (segment (start 114.185001 86.150001) (end 111.849999 86.150001) (width 0.25) (layer B.Cu) (net 25))
+  (segment (start 114.250001 86.085001) (end 114.185001 86.150001) (width 0.25) (layer B.Cu) (net 25))
+  (segment (start 114.250001 84.039999) (end 114.250001 86.085001) (width 0.25) (layer B.Cu) (net 25))
+  (segment (start 113.139999 83.649999) (end 113.860001 83.649999) (width 0.25) (layer B.Cu) (net 25))
+  (segment (start 113.389998 83.4) (end 113.139999 83.649999) (width 0.25) (layer B.Cu) (net 25))
+  (segment (start 113.5 83.4) (end 113.389998 83.4) (width 0.25) (layer B.Cu) (net 25))
+  (via (at 111.8 86.2) (size 0.8) (drill 0.4) (layers F.Cu B.Cu) (net 25))
+  (segment (start 113.860001 83.649999) (end 114.250001 84.039999) (width 0.25) (layer B.Cu) (net 25))
+  (segment (start 110.18 86.2) (end 110.11 86.13) (width 0.25) (layer F.Cu) (net 25))
+  (segment (start 111.8 86.2) (end 110.18 86.2) (width 0.25) (layer F.Cu) (net 25))
   (segment (start 111.137341 85.337339) (end 111.53734 84.93734) (width 0.25) (layer F.Cu) (net 24))
   (via (at 111.53734 84.93734) (size 0.8) (drill 0.4) (layers F.Cu B.Cu) (net 24))
@@
   (segment (start 113.5 84.4) (end 112.07468 84.4) (width 0.25) (layer B.Cu) (net 24))
   (segment (start 112.07468 84.4) (end 111.53734 84.93734) (width 0.25) (layer B.Cu) (net 24))
-  (segment (start 113.5 82.4) (end 112.89896 82.4) (width 0.25) (layer F.Cu) (net 25))
-  (segment (start 111.455001 87.125001) (end 111.16 86.83) (width 0.25) (layer F.Cu) (net 25))
-  (segment (start 111.948001 87.125001) (end 111.455001 87.125001) (width 0.25) (layer F.Cu) (net 25))
-  (segment (start 112.525001 86.548001) (end 111.948001 87.125001) (width 0.25) (layer F.Cu) (net 25))
-  (segment (start 111.16 86.83) (end 110.11 86.83) (width 0.25) (layer F.Cu) (net 25))
-  (segment (start 112.525001 82.773959) (end 112.525001 86.548001) (width 0.25) (layer F.Cu) (net 25))
-  (segment (start 112.89896 82.4) (end 112.525001 82.773959) (width 0.25) (layer F.Cu) (net 25))
-  (segment (start 101.91 96.135) (end 101.91 95.33) (width 0.25) (layer F.Cu) (net 26))
-  (segment (start 103.425 97.65) (end 101.91 96.135) (width 0.25) (layer F.Cu) (net 26))
-  (segment (start 103.425 98.55) (end 103.425 97.65) (width 0.25) (layer F.Cu) (net 26))
-  (segment (start 104.45 98.55) (end 111.375 98.55) (width 0.25) (layer F.Cu) (net 26))
-  (segment (start 103.425 98.55) (end 104.45 98.55) (width 0.25) (layer F.Cu) (net 26))
+  (segment (start 113.5 82.4) (end 112.89896 82.4) (width 0.25) (layer F.Cu) (net 26))
+  (segment (start 111.455001 87.125001) (end 111.16 86.83) (width 0.25) (layer F.Cu) (net 26))
+  (segment (start 111.948001 87.125001) (end 111.455001 87.125001) (width 0.25) (layer F.Cu) (net 26))
+  (segment (start 112.525001 86.548001) (end 111.948001 87.125001) (width 0.25) (layer F.Cu) (net 26))
+  (segment (start 111.16 86.83) (end 110.11 86.83) (width 0.25) (layer F.Cu) (net 26))
+  (segment (start 112.525001 82.773959) (end 112.525001 86.548001) (width 0.25) (layer F.Cu) (net 26))
+  (segment (start 112.89896 82.4) (end 112.525001 82.773959) (width 0.25) (layer F.Cu) (net 26))
+  (segment (start 101.91 96.135) (end 101.91 95.33) (width 0.25) (layer F.Cu) (net 23))
+  (segment (start 103.425 97.65) (end 101.91 96.135) (width 0.25) (layer F.Cu) (net 23))
+  (segment (start 103.425 98.55) (end 103.425 97.65) (width 0.25) (layer F.Cu) (net 23))
+  (segment (start 104.45 98.55) (end 111.375 98.55) (width 0.25) (layer F.Cu) (net 23))
+  (segment (start 103.425 98.55) (end 104.45 98.55) (width 0.25) (layer F.Cu) (net 23))
 )
