File: display.kicad_pcb (KiCad board)
At the start: 2 copper layers, 18.8 x 27.9 mm, 14 parts, among them J1 Conn_02x06_Counter_Clockwise, J2 Conn_01x05_Female, J3 Conn_01x02_Female, SW1 SW_Push, U1 MDBT42Q

Commit message: label tweaks
Other:
- board text added: "Copyright (c) 2018 Bobby D"
Changed lines of the file:
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@@
   (general
     (thickness 0.8)
-    (drawings 13)
+    (drawings 14)
     (tracks 209)
     (zones 0)
@@
     )
   )
+  (gr_text "Copyright (c) 2018 Bobby D" (at 106.9 104.3) (layer B.SilkS)
+    (effects (font (size 0.6 0.6) (thickness 0.1)) (justify mirror))
+  )
   (gr_text 3V3 (at 116.6 89.2 90) (layer F.SilkS)
